File: Hardware/Shifting_microSD.sch (EAGLE design)
At the start: 20 parts, among them U1 TXB0104, U2 3.3V

Commit message: updated version number for production
Other:
- note added: "v10"
- note removed: "v02"
Changed lines of the file:
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@@
 <plain>
 <text x="166.116" y="11.43" size="2.54" layer="94">Brent Wilkins</text>
-<text x="236.22" y="7.62" size="2.54" layer="94" font="vector">v02</text>
+<text x="236.22" y="7.62" size="2.54" layer="94" font="vector">v10</text>
 <text x="121.92" y="172.72" size="1.778" layer="97" font="vector" ratio="15" align="center">VCC +3.3V to +5.0V
 EXPECT UP TO VCC ON SIGNAL LINES</text>
