File: Production/Shifting_microSD_Panel_v10.brd (EAGLE design)
At the start: 122.9 x 259.6 mm, 1143 parts, among them U1 TXB0104, U10 TXB0104, U100 TXB0104, U101 3.3V, U102 TXB0104, U103 3.3V, U104 TXB0104, U105 3.3V, U106 TXB0104, U107 3.3V, U108 TXB0104, U109 3.3V, U11 3.3V, U110 TXB0104, U111 3.3V, U112 TXB0104, U113 3.3V, U114 TXB0104, U115 3.3V, U116 TXB0104, U117 3.3V, U118 TXB0104, U119 3.3V, U12 TXB0104, U120 TXB0104, U13 3.3V, U14 TXB0104, U15 3.3V, U16 TXB0104, U17 3.3V, U18 TXB0104, U19 3.3V, U2 3.3V, U20 TXB0104, U21 3.3V, U22 TXB0104, U23 3.3V, U24 TXB0104, U25 3.3V, U26 TXB0104, U27 3.3V, U28 TXB0104, U29 3.3V, U3 3.3V, U30 TXB0104, U31 3.3V, U32 TXB0104, U33 3.3V, U34 TXB0104, U35 3.3V, U36 TXB0104, U37 3.3V, U38 TXB0104, U39 3.3V, U4 TXB0104, U40 TXB0104, U41 3.3V, U42 TXB0104, U43 3.3V, U44 TXB0104, U45 3.3V, U46 TXB0104, U47 3.3V, U48 TXB0104, U49 3.3V, U5 3.3V, U50 TXB0104, U51 3.3V, U52 TXB0104, U53 3.3V, U54 TXB0104, U55 3.3V, U56 TXB0104, U57 3.3V, U58 TXB0104, U59 3.3V, U6 TXB0104, U60 TXB0104, U61 3.3V, U62 TXB0104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

Commit message: added bottom side panel fiducials
Parts:
- added E$3: (no value), SparkFun-Retired:FIDUCIAL-1.5X3
- added E$5, E$6: (no value), SparkFun-Aesthetics:FIDUCIAL-1X2
Changed lines of the file:
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@@
 <layer number="49" name="Reference" color="3" fill="1" visible="yes" active="yes"/>
 <layer number="50" name="dxf" color="7" fill="1" visible="yes" active="yes"/>
-<layer number="51" name="tDocu" color="6" fill="1" visible="no" active="yes"/>
+<layer number="51" name="tDocu" color="6" fill="1" visible="yes" active="yes"/>
 <layer number="52" name="bDocu" color="7" fill="1" visible="yes" active="yes"/>
 <layer number="53" name="tGND_GNDA" color="7" fill="9" visible="no" active="no"/>
@@
 <element name="E$1" library="SparkFun-Aesthetics" package="FIDUCIAL-1X2" value="" x="117.602" y="13.081" rot="R90"/>
 <element name="E$2" library="SparkFun-Retired" package="FIDUCIAL-1.5X3" value="" x="4.572" y="14.732"/>
+<element name="E$3" library="SparkFun-Retired" package="FIDUCIAL-1.5X3" value="" x="4.572" y="14.732" rot="MR0"/>
+<element name="E$5" library="SparkFun-Aesthetics" package="FIDUCIAL-1X2" value="" x="117.602" y="13.081" rot="MR90"/>
+<element name="E$6" library="SparkFun-Aesthetics" package="FIDUCIAL-1X2" value="" x="117.602" y="245.237" rot="MR90"/>
 </elements>
 <signals>
